File: KiCad/Keithley_20ChanSSR/Keithley_20ChanSSR.sch (KiCad schematic (older format))
At the start: 77 parts, among them J1 Screw_Terminal_01x10, J2 Screw_Terminal_01x12, J3 Conn_02x16_Top_Bottom, J4 Screw_Terminal_01x10, J5 Screw_Terminal_01x12, U1 TLP3558, U10 TLP3558, U11 TLP3558, U12 TLP3558, U13 TLP3558, U14 TLP3558, U15 TLP3558, U16 TLP3558, U17 TLP3558, U18 TLP3558, U19 TLP3558, U2 TLP3558, U20 TLP3558, U21 TLP3558, U22 TLP3558, U23 TLP3558, U24 TLP3558, U25 Arduino_Micro, U26 TLP3558, U27 TLP3558, U28 TLP3558, U29 TLP3558, U3 TLP3558, U30 TLP3558, U31 TLP3558, U32 TLP3558, U33 TLP3558, U34 TLP3558, U35 TLP3558, U36 TLP3558, U37 TLP3558, U38 TLP3558, U39 TLP3558, U4 TLP3558, U40 TLP3558, U41 TLP3558, U42 TLP3558, U43 TLP3558, U44 TLP3558, U45 TLP3558, U5 TLP3558, U6 TLP3558, U7 TLP3558, U8 TLP3558, U9 TLP3558

Commit message: Deleted some unused files, added the required library.
Parts:
- U1, U10, U11, U12, U13, U14, U15, U16, U17, U18, U19, U2, U20, U21, U22, U23, U24, U26, U27, U28, U29, U3, U30, U31, U32, U33, U34, U35, U36, U37, U38, U39, U4, U40, U41, U42, U43, U44, U45, U5, U6, U7, U8, U9: symbol CozKiCadLibrary:TLP3558 -> Keithley_20ChanSSR-rescue:TLP3558-CozKiCadLibrary
- U25: symbol CozKiCadLibrary:Arduino_Micro -> Keithley_20ChanSSR-rescue:Arduino_Micro-CozKiCadLibrary
Changed lines of the file:
@@
 $EndDescr
 $Comp
-L CozKiCadLibrary:TLP3558 U2
+L Keithley_20ChanSSR-rescue:TLP3558-CozKiCadLibrary U2
 U 1 1 5CD0E8BB
 P 6550 3800
@@
 $EndComp
 $Comp
-L CozKiCadLibrary:TLP3558 U11
+L Keithley_20ChanSSR-rescue:TLP3558-CozKiCadLibrary U11
 U 1 1 5CD919D7
 P 9750 3800
@@
 $EndComp
 $Comp
-L CozKiCadLibrary:TLP3558 U12
+L Keithley_20ChanSSR-rescue:TLP3558-CozKiCadLibrary U12
 U 1 1 5CD919E1
 P 10100 3800
@@
 $EndComp
 $Comp
-L CozKiCadLibrary:TLP3558 U13
+L Keithley_20ChanSSR-rescue:TLP3558-CozKiCadLibrary U13
 U 1 1 5CD919EB
 P 10450 3800
@@
 $EndComp
 $Comp
-L CozKiCadLibrary:TLP3558 U14
+L Keithley_20ChanSSR-rescue:TLP3558-CozKiCadLibrary U14
 U 1 1 5CD919F5
 P 10800 3800
@@
 $EndComp
 $Comp
-L CozKiCadLibrary:TLP3558 U15
+L Keithley_20ChanSSR-rescue:TLP3558-CozKiCadLibrary U15
 U 1 1 5CD919FF
 P 11150 3800
@@
 $EndComp
 $Comp
-L CozKiCadLibrary:TLP3558 U16
+L Keithley_20ChanSSR-rescue:TLP3558-CozKiCadLibrary U16
 U 1 1 5CD91A09
 P 11500 3800
@@
 $EndComp
 $Comp
-L CozKiCadLibrary:TLP3558 U17
+L Keithley_20ChanSSR-rescue:TLP3558-CozKiCadLibrary U17
 U 1 1 5CD91A13
 P 11850 3800
@@
 $EndComp
 $Comp
-L CozKiCadLibrary:TLP3558 U18
+L Keithley_20ChanSSR-rescue:TLP3558-CozKiCadLibrary U18
 U 1 1 5CD91A1D
 P 12200 3800
@@
 $EndComp
 $Comp
-L CozKiCadLibrary:TLP3558 U19
+L Keithley_20ChanSSR-rescue:TLP3558-CozKiCadLibrary U19
 U 1 1 5CD91A27
 P 12550 3800
@@
 $EndComp
 $Comp
-L CozKiCadLibrary:TLP3558 U20
+L Keithley_20ChanSSR-rescue:TLP3558-CozKiCadLibrary U20
 U 1 1 5D2A594A
 P 12900 3800
@@
 $EndComp
 $Comp
-L CozKiCadLibrary:TLP3558 U9
+L Keithley_20ChanSSR-rescue:TLP3558-CozKiCadLibrary U9
 U 1 1 5CF08C9D
 P 9000 3800
@@
 $EndComp
 $Comp
-L CozKiCadLibrary:TLP3558 U10
+L Keithley_20ChanSSR-rescue:TLP3558-CozKiCadLibrary U10
 U 1 1 5CD1F434
 P 9350 3800
@@
 $EndComp
 $Comp
-L CozKiCadLibrary:TLP3558 U7
+L Keithley_20ChanSSR-rescue:TLP3558-CozKiCadLibrary U7
 U 1 1 5CD1E31D
 P 8300 3800
@@
 $EndComp
 $Comp
-L CozKiCadLibrary:TLP3558 U8
+L Keithley_20ChanSSR-rescue:TLP3558-CozKiCadLibrary U8
 U 1 1 5CD1D556
 P 8650 3800
@@
 $EndComp
 $Comp
-L CozKiCadLibrary:TLP3558 U5
+L Keithley_20ChanSSR-rescue:TLP3558-CozKiCadLibrary U5
 U 1 1 5CD1C426
 P 7600 3800
@@
 $EndComp
 $Comp
-L CozKiCadLibrary:TLP3558 U6
+L Keithley_20ChanSSR-rescue:TLP3558-CozKiCadLibrary U6
 U 1 1 5CD1B8B7
 P 7950 3800
@@
 $EndComp
 $Comp
-L CozKiCadLibrary:TLP3558 U3
+L Keithley_20ChanSSR-rescue:TLP3558-CozKiCadLibrary U3
 U 1 1 5CD1B2F0
 P 6900 3800
@@
 $EndComp
 $Comp
-L CozKiCadLibrary:TLP3558 U4
+L Keithley_20ChanSSR-rescue:TLP3558-CozKiCadLibrary U4
 U 1 1 5CD1A77C
 P 7250 3800
@@
 $EndComp
 $Comp
-L CozKiCadLibrary:TLP3558 U26
+L Keithley_20ChanSSR-rescue:TLP3558-CozKiCadLibrary U26
 U 1 1 5D682CBB
 P 6200 5550
@@
 $EndComp
 $Comp
-L CozKiCadLibrary:TLP3558 U36
+L Keithley_20ChanSSR-rescue:TLP3558-CozKiCadLibrary U36
 U 1 1 5D682CC1
 P 9750 5550
@@
 $EndComp
 $Comp
-L CozKiCadLibrary:TLP3558 U37
+L Keithley_20ChanSSR-rescue:TLP3558-CozKiCadLibrary U37
 U 1 1 5D682CC7
 P 10100 5550
@@
 $EndComp
 $Comp
-L CozKiCadLibrary:TLP3558 U38
+L Keithley_20ChanSSR-rescue:TLP3558-CozKiCadLibrary U38
 U 1 1 5D682CCD
 P 10450 5550
@@
 $EndComp
 $Comp
-L CozKiCadLibrary:TLP3558 U39
+L Keithley_20ChanSSR-rescue:TLP3558-CozKiCadLibrary U39
 U 1 1 5D682CD3
 P 10800 5550
@@
 $EndComp
 $Comp
-L CozKiCadLibrary:TLP3558 U40
+L Keithley_20ChanSSR-rescue:TLP3558-CozKiCadLibrary U40
 U 1 1 5D682CD9
 P 11150 5550
@@
 $EndComp
 $Comp
-L CozKiCadLibrary:TLP3558 U41
+L Keithley_20ChanSSR-rescue:TLP3558-CozKiCadLibrary U41
 U 1 1 5D682CDF
 P 11500 5550
@@
 $EndComp
 $Comp
-L CozKiCadLibrary:TLP3558 U42
+L Keithley_20ChanSSR-rescue:TLP3558-CozKiCadLibrary U42
 U 1 1 5D682CE5
 P 11850 5550
@@
 $EndComp
 $Comp
-L CozKiCadLibrary:TLP3558 U43
+L Keithley_20ChanSSR-rescue:TLP3558-CozKiCadLibrary U43
 U 1 1 5D682CEB
 P 12200 5550
@@
 $EndComp
 $Comp
-L CozKiCadLibrary:TLP3558 U44
+L Keithley_20ChanSSR-rescue:TLP3558-CozKiCadLibrary U44
 U 1 1 5D682CF1
 P 12550 5550
@@
 	11950 5250 12100 5250
 $Comp
-L CozKiCadLibrary:TLP3558 U45
+L Keithley_20ChanSSR-rescue:TLP3558-CozKiCadLibrary U45
 U 1 1 5D682D0A
 P 12900 5550
@@
 	6300 5250 6450 5250
 $Comp
-L CozKiCadLibrary:TLP3558 U35
+L Keithley_20ChanSSR-rescue:TLP3558-CozKiCadLibrary U35
 U 1 1 5D682D65
 P 9350 5550
@@
 $EndComp
 $Comp
-L CozKiCadLibrary:TLP3558 U34
+L Keithley_20ChanSSR-rescue:TLP3558-CozKiCadLibrary U34
 U 1 1 5D682D6B
 P 9000 5550
@@
 $EndComp
 $Comp
-L CozKiCadLibrary:TLP3558 U33
+L Keithley_20ChanSSR-rescue:TLP3558-CozKiCadLibrary U33
 U 1 1 5D682D71
 P 8650 5550
@@
 $EndComp
 $Comp
-L CozKiCadLibrary:TLP3558 U32
+L Keithley_20ChanSSR-rescue:TLP3558-CozKiCadLibrary U32
 U 1 1 5D682D77
 P 8300 5550
@@
 $EndComp
 $Comp
-L CozKiCadLibrary:TLP3558 U31
+L Keithley_20ChanSSR-rescue:TLP3558-CozKiCadLibrary U31
 U 1 1 5D682D7D
 P 7950 5550
@@
 $EndComp
 $Comp
-L CozKiCadLibrary:TLP3558 U30
+L Keithley_20ChanSSR-rescue:TLP3558-CozKiCadLibrary U30
 U 1 1 5D682D83
 P 7600 5550
@@
 $EndComp
 $Comp
-L CozKiCadLibrary:TLP3558 U29
+L Keithley_20ChanSSR-rescue:TLP3558-CozKiCadLibrary U29
 U 1 1 5D682D89
 P 7250 5550
@@
 $EndComp
 $Comp
-L CozKiCadLibrary:TLP3558 U28
+L Keithley_20ChanSSR-rescue:TLP3558-CozKiCadLibrary U28
 U 1 1 5D682D8F
 P 6900 5550
@@
 $EndComp
 $Comp
-L CozKiCadLibrary:TLP3558 U27
+L Keithley_20ChanSSR-rescue:TLP3558-CozKiCadLibrary U27
 U 1 1 5D682D95
 P 6550 5550
@@
 	9250 6250 9250 6650
 $Comp
-L CozKiCadLibrary:TLP3558 U23
+L Keithley_20ChanSSR-rescue:TLP3558-CozKiCadLibrary U23
 U 1 1 5DCF3BF0
 P 13600 5350
@@
 $EndComp
 $Comp
-L CozKiCadLibrary:TLP3558 U24
+L Keithley_20ChanSSR-rescue:TLP3558-CozKiCadLibrary U24
 U 1 1 5DCF3BFA
 P 13950 5350
@@
 	6300 4100 6450 4100
 $Comp
-L CozKiCadLibrary:TLP3558 U1
+L Keithley_20ChanSSR-rescue:TLP3558-CozKiCadLibrary U1
 U 1 1 5CD19EF0
 P 6200 3800
@@
 Connection ~ 13200 3400
 $Comp
-L CozKiCadLibrary:TLP3558 U22
+L Keithley_20ChanSSR-rescue:TLP3558-CozKiCadLibrary U22
 U 1 1 5DB9136F
 P 13950 4450
@@
 Connection ~ 13200 5750
 $Comp
-L CozKiCadLibrary:TLP3558 U21
+L Keithley_20ChanSSR-rescue:TLP3558-CozKiCadLibrary U21
 U 1 1 5DB91365
 P 13600 4450
@@
 CLK
 $Comp
-L CozKiCadLibrary:Arduino_Micro U25
+L Keithley_20ChanSSR-rescue:Arduino_Micro-CozKiCadLibrary U25
 U 1 1 5D44B2E9
 P 3200 7150

Commit message: Cleaned up the schematic for better readibility
Parts:
- R1, R10, R11, R12, R13, R14, R15, R16, R17, R18, R19, R2, R20, R21, R22, R24, R3, R4, R5, R6, R7, R8, R9: value R -> 120R
- R23, R25, R26: value R -> 1K
Connections:
- net INPUT_LO: now also J2.11 (Pin_11), U1.3, U11.3, U13.3, U15.3, U17.3, U19.3, U21.3, U3.3, U5.3, U7.3, U9.3
- net SENSE_HI: now also J5.12 (Pin_12), U24.4
Other:
- note added: "20x \nTLP3558A"
- note added: "2x \nTLP3558A"
